Commit message: Gmapping is working sort-of well.

File: yertle.urdf (robot description, URDF)
Before this commit: robot test_robot, 7 links, 6 joints
Joints:
- joint base_to_kinect: origin xyz=0.0 0 0.22 rpy=0 0 0 -> xyz=0.12 0 0.20 rpy=0 0 0

Commit message: Lots of changes

File: yertle.urdf (robot description, URDF)
Before this commit: robot test_robot, 7 links, 6 joints
Links:
- added link range0; visual box size=0.01 0.03 0.005
- added link range1; visual box size=0.01 0.03 0.005
- added link range2; visual box size=0.01 0.03 0.005
- link base_link: geometry visual cylinder length=0.01 radius=0.21
Joints:
- added joint base_to_range0: type fixed, parent base_link, child range0, origin xyz=0.1414 -0.1414 0.085 rpy=0 0 -0.7854
- added joint base_to_range1: type fixed, parent base_link, child range1, origin xyz=0.20 0 0.085 rpy=0 0 0
- added joint base_to_range2: type fixed, parent base_link, child range2, origin xyz=0.1414 0.1414 0.085 rpy=0 0 0.7854
